File: ECAD/PCBs/ABSIS/ABSIS_ALE+/ABSIS ALE+.kicad_sch (KiCad schematic)
At the start: 48 parts, among them IC1 THVD1410DR, IC2 TPS563300DRLR, J1 39-28-8060, J11 2.54-2*2P, J12 PZ254V-11-03P, J2 39-28-8060, J3 PZ254V-11-02P, J4 PZ254V-11-03P, J5 PZ254V-11-02P, J6 B2B-XH-A(LF)(SN), J7 B2B-XH-A(LF)(SN), J8 B-2100S12P-B110, J9 B-2100S12P-B110, Q1 AO3400A, Q2 IRLML6402TRPBF, Q3 AO3400A, Q4 IRLML6402TRPBF

Commit message: Partial ALE+ work
Connections:
- net FB(TPS): no longer names the net of C7.2, IC2.8 (FB), R11.2, R12.1
Other:
- note removed: "ABSIS BUS CONNECTORS"
- note removed: "MOUNTING HOLES"
- moved on the sheet: C2, C3, C4, C5, C6, C7, C8, D2, D3, F1, H1, H2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
