File: ECAD/PCBs/ABSIS/ABSIS_OH_Micro/ABSIS_OH_Micro.kicad_pcb (KiCad board)
At the start: 4 copper layers, 17.8 x 41 mm, 42 parts, among them CN1 M12PTH, CN2 M12PTH, J2 DX07S016JA1R1500, U1 MIC5219, U2 TPS2116DRL, U3 USBLC6-2SC6, U4 REF3040, U5 ATmega32U4-M, Y2 16MHz

Commit message: New OH_Micro Start
Parts:
- removed C10: 10uF, Capacitor_Tantalum_SMD:CP_EIA-3216-18_Kemet-A
- added C18: 0.1uF, Capacitor_SMD:C_0402_1005Metric, F.Cu at (144.0, 113.8)
- added C19: 0.1uF, Capacitor_SMD:C_0402_1005Metric, F.Cu at (149.1, 105.6)
- added C20: 0.1uF, Capacitor_SMD:C_0402_1005Metric, F.Cu at (149.6, 116.6)
- added C21: 1uF, Capacitor_SMD:C_0402_1005Metric, F.Cu at (146.8, 105.5)
- added C6: 10uF, Capacitor_SMD:C_0402_1005Metric, F.Cu at (155.9, 90.5)
- added C7: 22uF, Capacitor_SMD:C_0805_2012Metric, F.Cu at (149.4, 93.3)
- added FB1: FerriteBead_Small, Inductor_SMD:L_0402_1005Metric, F.Cu at (148.7, 103.6)
- added R13: 10K, Resistor_SMD:R_0402_1005Metric, F.Cu at (148.6, 94.9)
- added RST1: RST, OH_Footprints:SolderJumper-2_P1.3mm_Open_RoundedPad1.0x1.5mm, B.Cu at (116.5, 100.3)
- C11: value 1uF -> 0.1uF; footprint Capacitor_SMD:C_0603_1608Metric -> Capacitor_SMD:C_0402_1005Metric
- C12, C13, C16, C17, C3, C4, C5: footprint Capacitor_SMD:C_0603_1608Metric -> Capacitor_SMD:C_0402_1005Metric
- C14, C15: value 22pF -> 12pF; footprint Capacitor_SMD:C_0603_1608Metric -> Capacitor_SMD:C_0402_1005Metric
- D1, D5: footprint LED_SMD:LED_0603_1608Metric -> LED_SMD:LED_0402_1005Metric
- R1, R11, R12, R2, R3, R6: footprint Resistor_SMD:R_0603_1608Metric -> Resistor_SMD:R_0402_1005Metric
- R10: footprint Resistor_SMD:R_0201_0603Metric -> Resistor_SMD:R_0402_1005Metric
- R4, R5: footprint OH_Footprints:R_0603_1608Metric -> Resistor_SMD:R_0402_1005Metric
- R7: value 15k -> 36K; footprint Resistor_SMD:R_0603_1608Metric -> Resistor_SMD:R_0402_1005Metric
- R8: value 4K7 -> 10K; footprint Resistor_SMD:R_0603_1608Metric -> Resistor_SMD:R_0402_1005Metric
- R9: value 4K7 -> 470K; footprint Resistor_SMD:R_0603_1608Metric -> Resistor_SMD:R_0402_1005Metric
- Y2: footprint Crystal:Crystal_SMD_TXC_7A-2Pin_5x3.2mm -> Crystal:Crystal_SMD_3225-4Pin_3.2x2.5mm
- moved R9 38.7 mm to (148.6, 95.9), turned to 180 degrees
- moved R8 35.9 mm to (148.6, 96.9), turned to 180 degrees
- moved R7 35.3 mm to (151.0, 97.6), turned to 180 degrees
- moved U2 34.6 mm to (151.0, 95.7)
- moved U4 24.6 mm to (152.0, 103.6), turned to 90 degrees
- moved R11 23.0 mm to (143.0, 122.1), turned to 180 degrees
- moved C5 23.0 mm to (149.7, 103.6), turned to -90 degrees
- moved D1 21.6 mm to (141.0, 122.1), turned to 180 degrees
- moved R10 12.4 mm to (131.2, 105.1), turned to -135 degrees
- moved R12 12.0 mm to (154.2, 122.2)
- moved R4 9.96 mm to (145.4, 106.9), turned to -45 degrees
- moved R5 8.85 mm to (146.1, 106.2), turned to -45 degrees
- moved C12 8.67 mm to (144.7, 108.2), turned to -135 degrees
- moved D5 7.34 mm to (156.1, 122.2)
- moved C13 7.28 mm to (150.4, 106.9), turned to -45 degrees
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Connections:
- R9 pad 1: +5V -> /PR1
- R9 pad 2: /D30 -> /ST
- U2 pad 5: /PR1 -> /VIN1
- U2 pad 8: /D30 -> /ST
- U5 pad 24: +5V -> /AVCC
- U5 pad 33: GND -> unconnected-(U5-~{HWB}/PE2-Pad33)
- U5 pad 44: +5V -> /AVCC
- Y2 pad 2: /XTAL1 -> GND
Routing:
- added copper zone on In1.Cu, net GND
- added copper zone on In2.Cu, net GND
